File: layout/arduino-nano/ArduinoSpecAn.sch (KiCad schematic (older format))
At the start: 46 parts, among them J1 SMA, J2 SMA, P1 CONN_01X08, P2 CONN_01X06, P3 CONN_01X08, Q1 MMBT3904, Q2 MMBT3904, U1 AD8307, U2 AD9851, U3 LM7301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

Commit message: Working on layout
Parts:
- J1: footprint (none) -> footprints:SMA_Edgemount
- gave numbers to parts that had none: 1
Changed lines of the file:
@@
 	-2350 5550 -2300 5550
 $Comp
-L MCU_Module:Arduino_Nano_v3.x A?
+L MCU_Module:Arduino_Nano_v3.x A1
 U 1 1 5B672321
 P 2100 2250
-F 0 "A?" H 2100 1164 50  0000 C CNN
+F 0 "A1" H 2100 1164 50  0000 C CNN
 F 1 "Arduino_Nano_v3.x" H 2100 1073 50  0000 C CNN
 F 2 "Module:Arduino_Nano" H 2250 1300 50  0001 L CNN
@@
 $EndComp
 $Comp
-L power:GND #PWR?
+L power:GND #PWR0101
 U 1 1 5B67284E
 P 2150 3550
-F 0 "#PWR?" H 2150 3300 50  0001 C CNN
+F 0 "#PWR0101" H 2150 3300 50  0001 C CNN
 F 1 "GND" H 2155 3377 50  0000 C CNN
 F 2 "" H 2150 3550 50  0001 C CNN
@@
 	2400 1250 2400 1100
 $Comp
-L power:+3V3 #PWR?
+L power:+3V3 #PWR0102
 U 1 1 5B6A5A5B
 P 2100 1100
-F 0 "#PWR?" H 2100 950 50  0001 C CNN
+F 0 "#PWR0102" H 2100 950 50  0001 C CNN
 F 1 "+3V3" H 2115 1273 50  0000 C CNN
 F 2 "" H 2100 1100 50  0001 C CNN
@@
 $EndComp
 $Comp
-L power:+5V #PWR?
+L power:+5V #PWR0103
 U 1 1 5B6A5B31
 P 2400 1100
-F 0 "#PWR?" H 2400 950 50  0001 C CNN
+F 0 "#PWR0103" H 2400 950 50  0001 C CNN
 F 1 "+5V" H 2415 1273 50  0000 C CNN
 F 2 "" H 2400 1100 50  0001 C CNN
@@
 Wire Notes Line
 	3400 3550 3400 600
-$Comp
-L ArduinoSpecAn-rescue:SMA J1
-U 1 1 5B70300F
-P 6000 950
-F 0 "J1" H 5762 897 60  0000 R CNN
-F 1 "SMA" H 5762 791 60  0000 R CNN
-F 2 "" H 6000 950 60  0000 C CNN
-F 3 "" H 6000 950 60  0000 C CNN
-	1    6000 950
-	-1   0    0    -1
-$EndComp
 Text Label 2850 2250 2    60   ~ 0
 A0
@@
 	-8750 -650 -8650 -650
 $Comp
-L power:GND #PWR?
+L power:GND #PWR0104
 U 1 1 5B7475F9
 P 9350 1500
-F 0 "#PWR?" H 9350 1250 50  0001 C CNN
+F 0 "#PWR0104" H 9350 1250 50  0001 C CNN
 F 1 "GND" H 9350 1350 50  0000 C CNN
 F 2 "" H 9350 1500 60  0000 C CNN
@@
 Text Label -8750 -1250 0    60   ~ 0
 5V
+$Comp
+L ArduinoSpecAn-rescue:SMA J1
+U 1 1 5B7B44E1
+P 6000 950
+F 0 "J1" H 5750 850 60  0000 C CNN
+F 1 "SMA" H 6000 1150 60  0000 C CNN
+F 2 "footprints:SMA_Edgemount" H 6000 950 60  0001 C CNN
+F 3 "" H 6000 950 60  0000 C CNN
+	1    6000 950
+	-1   0    0    -1
+$EndComp
 $EndSCHEMATC

Commit message: Removed DDS
Parts:
- removed C1: .01uF, footprints:Custom_0805, symbol ArduinoSpecAn-rescue:C_Small
- removed C10, C7: 10pF, footprints:Custom_0805, symbol ArduinoSpecAn-rescue:C_Small
- removed C11, C12, C13, C14: .1uF, footprints:Custom_0805, symbol ArduinoSpecAn-rescue:C_Small
- removed C3, C6: 10uF, footprints:Custom_0805, symbol ArduinoSpecAn-rescue:C_Small
- removed C8, C9: 39pF, footprints:Custom_0805, symbol ArduinoSpecAn-rescue:C_Small
- removed L1, L3: 270nH, footprints:Custom_0805, symbol ArduinoSpecAn-rescue:L_Small
- removed L2: 470nH, footprints:Custom_0805, symbol ArduinoSpecAn-rescue:L_Small
- removed P1, P3: CONN_01X08, Pin_Headers:Pin_Header_Straight_1x08, symbol ArduinoSpecAn-rescue:CONN_01X08
- removed P2: CONN_01X06, Pin_Headers:Pin_Header_Straight_1x06, symbol ArduinoSpecAn-rescue:CONN_01X06
- removed Pot1: 1k, footprints:ST4ETB_Trim_Pot, symbol ArduinoSpecAn-rescue:POT
- removed Q1, Q2: MMBT3904, footprints:SOT-23, symbol ArduinoSpecAn-rescue:MMBT3904
- removed R1: 3k92, footprints:Custom_0805, symbol ArduinoSpecAn-rescue:R_Small
- removed R10, R13, R4: 100, footprints:Custom_0805, symbol ArduinoSpecAn-rescue:R_Small
- removed R14, R15: 2k, footprints:Custom_0805, symbol ArduinoSpecAn-rescue:R_Small
- removed R5, R6, R7: 220, footprints:Custom_0805, symbol ArduinoSpecAn-rescue:R_Small
- removed R8: 47, footprints:Custom_0805, symbol ArduinoSpecAn-rescue:R_Small
- removed R9: 50, footprints:Custom_0805, symbol ArduinoSpecAn-rescue:R_Small
- removed U2: AD9851, Housings_SSOP:SSOP-28_5.3x10.2mm_Pitch0.65mm, symbol ArduinoSpecAn-rescue:AD9851
- removed X1: KC5032A, footprints:KC5032A-CM_SMD_Crystal, symbol ArduinoSpecAn-rescue:KC5032A
- C15: value .1uF -> 100nF; footprint footprints:Custom_0805 -> Capacitor_SMD:C_0805_2012Metric_Pad1.15x1.50mm_HandSolder
- C2, C4, C5: footprint footprints:Custom_0805 -> Capacitor_SMD:C_0805_2012Metric_Pad1.15x1.50mm_HandSolder
- R11, R12: value 1k -> 1kΩ; footprint footprints:Custom_0805 -> Resistor_SMD:R_0805_2012Metric_Pad1.15x1.50mm_HandSolder
- R2: value 51 -> 51Ω; footprint footprints:Custom_0805 -> Resistor_SMD:R_0805_2012Metric_Pad1.15x1.50mm_HandSolder
- R3: footprint footprints:Custom_0805 -> Resistor_SMD:R_0805_2012Metric_Pad1.15x1.50mm_HandSolder
Connections:
- net 5V is gone; now on net +5V: C15.1, R3.2, U3.5 (V+)
- no-connect marks 24 -> 2
Other:
- note added: "Arduino"
- note removed: "50 Ohm output impedance.\nWill drive 0 dBm into 50 Ohm load."
- note removed: "72MHz Butterworth LPF\nMatched to 100 Ohms"
- note removed: "Decoupling Caps:\n- AD9851 x 4"
- moved on the sheet: C15, C2, C4, C5, J2, R11, R12, R2, R3, U1, U3
