File: layout/arduino-nano-AD9851/ArduinoSpecAn.sch (KiCad schematic (older format))
At the start: 45 parts, among them J1 SMA, J2 SMA, Q1 MMBT3904, Q2 MMBT3904, U1 AD8307, U2 AD9851, U3 LM7301, X1 KC5032A

Commit message: Mostly finished
Parts:
- added R16, R17: 1kΩ, Resistor_SMD:R_0805_2012Metric_Pad1.15x1.50mm_HandSolder, symbol Device:R
- C1: value .01uF -> 100nF; footprint footprints:Custom_0805 -> Capacitor_SMD:C_0805_2012Metric_Pad1.15x1.50mm_HandSolder
- C10, C7, C8, C9: footprint footprints:Custom_0805 -> Capacitor_SMD:C_0805_2012Metric_Pad1.15x1.50mm_HandSolder
- C11, C12, C13, C14, C15, C5: value .1uF -> 100nF; footprint footprints:Custom_0805 -> Capacitor_SMD:C_0805_2012Metric_Pad1.15x1.50mm_HandSolder
- C2, C3, C4, C6: value 10uF -> 10µF; footprint footprints:Custom_0805 -> Capacitor_SMD:C_0805_2012Metric_Pad1.15x1.50mm_HandSolder
- L1, L2, L3: footprint footprints:Custom_0805 -> Inductor_SMD:L_0805_2012Metric_Pad1.15x1.50mm_HandSolder
- Pot1: footprint footprints:ST4ETB_Trim_Pot -> Potentiometer_THT:Potentiometer_Piher_PT-10-V05_Vertical
- R1: value 3k92 -> 3.9kΩ; footprint footprints:Custom_0805 -> Resistor_SMD:R_0805_2012Metric_Pad1.15x1.50mm_HandSolder
- R10, R13, R4: value 100 -> 100Ω; footprint footprints:Custom_0805 -> Resistor_SMD:R_0805_2012Metric_Pad1.15x1.50mm_HandSolder
- R11, R12: value 1k -> 1kΩ; footprint footprints:Custom_0805 -> Resistor_SMD:R_0805_2012Metric_Pad1.15x1.50mm_HandSolder
- R14, R15: value 2k -> 2kΩ; footprint footprints:Custom_0805 -> Resistor_SMD:R_0805_2012Metric_Pad1.15x1.50mm_HandSolder
- R2: value 51 -> 51Ω; footprint footprints:Custom_0805 -> Resistor_SMD:R_0805_2012Metric_Pad1.15x1.50mm_HandSolder
- R3: value 4R7 -> 4.7Ω; footprint footprints:Custom_0805 -> Resistor_SMD:R_0805_2012Metric_Pad1.15x1.50mm_HandSolder
- R5, R6, R7: value 220 -> 220Ω; footprint footprints:Custom_0805 -> Resistor_SMD:R_0805_2012Metric_Pad1.15x1.50mm_HandSolder
- R8: value 47 -> 47Ω; footprint footprints:Custom_0805 -> Resistor_SMD:R_0805_2012Metric_Pad1.15x1.50mm_HandSolder
- R9: value 50 -> 50Ω; footprint footprints:Custom_0805 -> Resistor_SMD:R_0805_2012Metric_Pad1.15x1.50mm_HandSolder
Connections:
- net GND: now also D1.2 (A), D2.2 (A)
- net at D1.1 (K): now also R16.2
- net at D2.1 (K): now also R17.2
- net A1: now reaches A1.20 (A1)
- net A1: now also R16.1
- net A2: now reaches A1.21 (A2)
- net A2: now also R17.1
