File: layout/arduino-nano-AD9851/ArduinoSpecAn.kicad_pcb (KiCad board)
At the start: 2 copper layers, 60.2 x 50.8 mm, 45 parts, among them J1 SMA, J2 SMA, Q1 MMBT3904, Q2 MMBT3904, U1 AD8307, U2 AD9851, U3 LM7301, X1 KC5032A

Commit message: Mostly finished
Parts:
- added R16: 1kΩ, Resistor_SMD:R_0805_2012Metric_Pad1.15x1.50mm_HandSolder, F.Cu at (110.2, 131.1)
- added R17: 1kΩ, Resistor_SMD:R_0805_2012Metric_Pad1.15x1.50mm_HandSolder, F.Cu at (110.2, 134.1)
- added REF**: OSHW-Logo_11.4x12mm_SilkScreen, Symbol:OSHW-Logo_11.4x12mm_SilkScreen, B.Cu at (158.8, 92.2)
- added REF**: WEEE-Logo_5.6x8mm_SilkScreen, Symbol:WEEE-Logo_5.6x8mm_SilkScreen, B.Cu at (158.5, 102.4)
- C1: value .01uF -> 100nF; footprint footprints:Custom_0805 -> Capacitor_SMD:C_0805_2012Metric_Pad1.15x1.50mm_HandSolder
- C10, C7, C8, C9: footprint footprints:Custom_0805 -> Capacitor_SMD:C_0805_2012Metric_Pad1.15x1.50mm_HandSolder
- C11, C12, C13, C14, C15, C5: value .1uF -> 100nF; footprint footprints:Custom_0805 -> Capacitor_SMD:C_0805_2012Metric_Pad1.15x1.50mm_HandSolder
- C2, C3, C4, C6: value 10uF -> 10µF; footprint footprints:Custom_0805 -> Capacitor_SMD:C_0805_2012Metric_Pad1.15x1.50mm_HandSolder
- L1, L2, L3: footprint footprints:Custom_0805 -> Inductor_SMD:L_0805_2012Metric_Pad1.15x1.50mm_HandSolder
- Pot1: footprint footprints:ST4ETB_Trim_Pot -> Potentiometer_THT:Potentiometer_Piher_PT-10-V05_Vertical
- R1: value 3k92 -> 3.9kΩ; footprint footprints:Custom_0805 -> Resistor_SMD:R_0805_2012Metric_Pad1.15x1.50mm_HandSolder
- R10, R13, R4: value 100 -> 100Ω; footprint footprints:Custom_0805 -> Resistor_SMD:R_0805_2012Metric_Pad1.15x1.50mm_HandSolder
- R11, R12: value 1k -> 1kΩ; footprint footprints:Custom_0805 -> Resistor_SMD:R_0805_2012Metric_Pad1.15x1.50mm_HandSolder
- R14, R15: value 2k -> 2kΩ; footprint footprints:Custom_0805 -> Resistor_SMD:R_0805_2012Metric_Pad1.15x1.50mm_HandSolder
- R2: value 51 -> 51Ω; footprint footprints:Custom_0805 -> Resistor_SMD:R_0805_2012Metric_Pad1.15x1.50mm_HandSolder
- R3: value 4R7 -> 4.7Ω; footprint footprints:Custom_0805 -> Resistor_SMD:R_0805_2012Metric_Pad1.15x1.50mm_HandSolder
- R5, R6, R7: value 220 -> 220Ω; footprint footprints:Custom_0805 -> Resistor_SMD:R_0805_2012Metric_Pad1.15x1.50mm_HandSolder
- R8: value 47 -> 47Ω; footprint footprints:Custom_0805 -> Resistor_SMD:R_0805_2012Metric_Pad1.15x1.50mm_HandSolder
- R9: value 50 -> 50Ω; footprint footprints:Custom_0805 -> Resistor_SMD:R_0805_2012Metric_Pad1.15x1.50mm_HandSolder
- moved R14 39.8 mm to (132.3, 114.0), turned to 90 degrees
- moved R15 34.3 mm to (128.5, 114.0), turned to 90 degrees
- moved D1 4.19 mm to (114.4, 131.1)
- moved D2 4.06 mm to (114.4, 134.1)
- moved Pot1 3.45 mm to (134.1, 94.0), turned to 0 degrees
Connections:
- A1 pad 20: (no net) -> /A1
- A1 pad 21: (no net) -> /A2
- D1 pad 1: (no net) -> Net-(D1-Pad1)
- D1 pad 2: (no net) -> GND
- D2 pad 1: (no net) -> Net-(D2-Pad1)
- D2 pad 2: (no net) -> GND
Routing:
- net /5V: track 61.3 -> 187.8 mm, vias 3 -> 7
- net /A0: track 3.13 -> 54.0 mm, vias 0 -> 1
- net /SLD: track 0.00 -> 49.4 mm, vias 0 -> 2
- net /SCL: track 0.00 -> 49.2 mm, vias 0 -> 2
- net /SDA: track 0.00 -> 42.2 mm
- net /A2: track 0.00 -> 33.4 mm, vias 0 -> 1
- net /A1: track 0.00 -> 32.8 mm, vias 0 -> 1
- net GND: track 163.4 -> 175.4 mm, vias 54 -> 59
- net Net-(Pot1-Pad3): track 0.00 -> 9.14 mm, vias 0 -> 2
- net (no net): track 0.00 -> 5.73 mm, vias 0 -> 2
- net Net-(Pot1-Pad2): track 9.29 -> 13.8 mm
- net Net-(D1-Pad1): track 0.00 -> 2.15 mm
- net Net-(D2-Pad1): track 0.00 -> 2.13 mm
- net Net-(C3-Pad2): track 6.77 -> 5.85 mm
Other:
- board text added: "Active"
- board text added: "Connected"
- board text added: "Network Analyzer Rev. 3b"
- board text added: "OpenNetworkAnalyzer Andreas Butti, 2018 https://github.com/andreasb242/OpenNetworkAnalyzer Based on https://hackaday.io/project/10021-arduino-network-analyzer"
- board text removed: "Arduino Uno Network Analyzer Shield Revision 2"
