File: layout/arduino-nano-SI5351/ArduinoSpecAn.sch (KiCad schematic (older format))
At the start: 35 parts, among them J1 SMA, J2 SMA, Q1 Q_NMOS_GSD, Q6 Q_NMOS_GSD, U1 AD8307, U2 LM1117-3.3, U3 LM7301, U4 SI5351, Y1 25MHz

Commit message: Mostly finished
Parts:
- R7, R8: value R -> 1kΩ
Connections:
- net GND: now also D1.1 (K), D2.1 (K); no longer R7.2, R8.2
- net at A1.8 (D5): no longer D1.1 (K)
- net at D1.2 (A): now also R7.2; no longer R7.1
- net at A1.7 (D4): no longer D2.1 (K)
- net at D2.2 (A): now also R8.2; no longer R8.1
- net A1: now reaches A1.20 (A1)
- net A1: now also R8.1
- net A2: now reaches A1.21 (A2)
- net A2: now also R7.1
- no-connect marks 2 -> 23
Other:
- moved on the sheet: D1, D2, R7, R8
Changed lines of the file:
@@
-$EndComp
-$Comp
-L power:GND #PWR02
-U 1 1 567B2AA5
-P 5200 1350
-F 0 "#PWR02" H 5200 1100 50  0001 C CNN
-F 1 "GND" H 5200 1200 50  0000 C CNN
-F 2 "" H 5200 1350 60  0000 C CNN
-F 3 "" H 5200 1350 60  0000 C CNN
-	1    5200 1350
-	1    0    0    -1
 $EndComp
 $Comp
@@
 $EndComp
 $Comp
-L power:GND #PWR03
-U 1 1 567B2DB3
-P 7500 1550
-F 0 "#PWR03" H 7500 1300 50  0001 C CNN
-F 1 "GND" H 7500 1400 50  0000 C CNN
-F 2 "" H 7500 1550 60  0000 C CNN
-F 3 "" H 7500 1550 60  0000 C CNN
-	1    7500 1550
-	1    0    0    -1
-$EndComp
-$Comp
 L ArduinoSpecAn-rescue:R_Small R3
 U 1 1 567B2F06
@@
 	5300 1950 5850 1950
 Wire Wire Line
-	7350 1450 7350 1500
-Wire Wire Line
-	7350 1500 7450 1500
-Wire Wire Line
-	7650 1500 7650 1450
-Wire Wire Line
-	7450 1450 7450 1500
-Connection ~ 7450 1500
-Wire Wire Line
-	7550 1450 7550 1500
-Connection ~ 7550 1500
-Wire Wire Line
-	7500 1550 7500 1500
-Connection ~ 7500 1500
-Wire Wire Line
 	6950 2050 6950 1850
 Connection ~ 6950 1850
-$Comp
-L power:GND #PWR012
-U 1 1 567C5089
-P 6950 2300
-F 0 "#PWR012" H 6950 2050 50  0001 C CNN
-F 1 "GND" H 6950 2150 50  0000 C CNN
-F 2 "" H 6950 2300 60  0000 C CNN
-F 3 "" H 6950 2300 60  0000 C CNN
-	1    6950 2300
-	1    0    0    -1
-$EndComp
-Wire Wire Line
-	6950 2300 6950 2250
 $Comp
 L ArduinoSpecAn-rescue:R_Small R12
@@
 Wire Wire Line
 	4550 1400 4700 1400
-Wire Wire Line
-	7450 1500 7500 1500
-Wire Wire Line
-	7550 1500 7650 1500
-Wire Wire Line
-	7500 1500 7550 1500
 Wire Wire Line
 	6950 1850 7150 1850
@@
 L Device:LED D1
 U 1 1 5B623ADF
-P 800 3300
-F 0 "D1" V 745 3378 50  0000 L CNN
-F 1 "LED" V 836 3378 50  0000 L CNN
-F 2 "LED_SMD:LED_0805_2012Metric_Pad0.97x1.50mm_HandSolder" H 800 3300 50  0001 C CNN
-F 3 "~" H 800 3300 50  0001 C CNN
-	1    800  3300
-	0    1    1    0
+P 3050 3900
+F 0 "D1" V 2995 3978 50  0000 L CNN
+F 1 "LED" V 3086 3978 50  0000 L CNN
+F 2 "LED_SMD:LED_0805_2012Metric_Pad0.97x1.50mm_HandSolder" H 3050 3900 50  0001 C CNN
+F 3 "~" H 3050 3900 50  0001 C CNN
+	1    3050 3900
+	0    -1   -1   0
 $EndComp
 $Comp
 L Device:R R7
 U 1 1 5B623D91
-P 800 3650
-F 0 "R7" H 870 3696 50  0000 L CNN
-F 1 "R" H 870 3605 50  0000 L CNN
-F 2 "Resistor_SMD:R_0805_2012Metric_Pad1.15x1.50mm_HandSolder" V 730 3650 50  0001 C CNN
-F 3 "~" H 800 3650 50  0001 C CNN
-	1    800  3650
+P 3050 3550
+F 0 "R7" H 3120 3596 50  0000 L CNN
+F 1 "1kΩ" H 3120 3505 50  0000 L CNN
+F 2 "Resistor_SMD:R_0805_2012Metric_Pad1.15x1.50mm_HandSolder" V 2980 3550 50  0001 C CNN
+F 3 "~" H 3050 3550 50  0001 C CNN
+	1    3050 3550
 	1    0    0    -1
 $EndComp
@@
 L Device:LED D2
 U 1 1 5B624246
-P 600 3300
-F 0 "D2" V 545 3378 50  0000 L CNN
-F 1 "LED" V 636 3378 50  0000 L CNN
-F 2 "LED_SMD:LED_0805_2012Metric_Pad0.97x1.50mm_HandSolder" H 600 3300 50  0001 C CNN
-F 3 "~" H 600 3300 50  0001 C CNN
-	1    600  3300
-	0    1    1    0
+P 2850 3900
+F 0 "D2" V 2795 3978 50  0000 L CNN
+F 1 "LED" V 2886 3978 50  0000 L CNN
+F 2 "LED_SMD:LED_0805_2012Metric_Pad0.97x1.50mm_HandSolder" H 2850 3900 50  0001 C CNN
+F 3 "~" H 2850 3900 50  0001 C CNN
+	1    2850 3900
+	0    -1   -1   0
 $EndComp
 $Comp
 L Device:R R8
 U 1 1 5B62424C
-P 600 3650
-F 0 "R8" H 670 3696 50  0000 L CNN
-F 1 "R" H 670 3605 50  0000 L CNN
-F 2 "Resistor_SMD:R_0805_2012Metric_Pad1.15x1.50mm_HandSolder" V 530 3650 50  0001 C CNN
-F 3 "~" H 600 3650 50  0001 C CNN
-	1    600  3650
-	1    0    0    -1
-$EndComp
-Wire Wire Line
-	600  3500 600  3450
-Wire Wire Line
-	800  3450 800  3500
-Wire Wire Line
-	600  3800 700  3800
+P 2850 3550
+F 0 "R8" H 2920 3596 50  0000 L CNN
+F 1 "1kΩ" H 2920 3505 50  0000 L CNN
+F 2 "Resistor_SMD:R_0805_2012Metric_Pad1.15x1.50mm_HandSolder" V 2780 3550 50  0001 C CNN
+F 3 "~" H 2850 3550 50  0001 C CNN
+	1    2850 3550
+	1    0    0    -1
+$EndComp
+Wire Wire Line
+	2850 3750 2850 3700
+Wire Wire Line
+	3050 3700 3050 3750
+Wire Wire Line
+	2850 4050 2950 4050
 $Comp
 L power:GND #PWR0113
 U 1 1 5B63FAE9
-P 700 3800
-F 0 "#PWR0113" H 700 3550 50  0001 C CNN
-F 1 "GND" H 705 3627 50  0000 C CNN
-F 2 "" H 700 3800 50  0001 C CNN
-F 3 "" H 700 3800 50  0001 C CNN
-	1    700  3800
-	1    0    0    -1
-$EndComp
-Connection ~ 700  3800
-Wire Wire Line
-	700  3800 800  3800
+P 2950 4050
+F 0 "#PWR0113" H 2950 3800 50  0001 C CNN
+F 1 "GND" H 2955 3877 50  0000 C CNN
+F 2 "" H 2950 4050 50  0001 C CNN
+F 3 "" H 2950 4050 50  0001 C CNN
+	1    2950 4050
+	1    0    0    -1
+$EndComp
+Connection ~ 2950 4050
+Wire Wire Line
+	2950 4050 3050 4050
 $Comp
 L MCU_Module:Arduino_Nano_v3.x A1
@@
 	1    0    0    -1
 $EndComp
-Wire Wire Line
-	750  3150 800  3150
-Wire Wire Line
-	600  3150 600  2050
-Wire Wire Line
-	600  2050 800  2050
-Wire Wire Line
-	800  2150 750  2150
-Wire Wire Line
-	750  2150 750  3150
+NoConn ~ 800  2950
+NoConn ~ 800  2850
+NoConn ~ 800  2750
+NoConn ~ 800  2650
+NoConn ~ 800  2550
+NoConn ~ 800  2450
+NoConn ~ 800  2350
+NoConn ~ 800  2250
+NoConn ~ 800  1650
+NoConn ~ 800  1750
+NoConn ~ 800  1850
+NoConn ~ 800  1950
+NoConn ~ 1800 1650
+NoConn ~ 1800 1750
+NoConn ~ 1800 2050
+NoConn ~ 1800 2550
+NoConn ~ 1200 1250
+NoConn ~ 1800 2850
+NoConn ~ 1800 2950
+$Comp
+L power:GND #PWR0114
+U 1 1 5B6974B6
+P 5200 1350
+F 0 "#PWR0114" H 5200 1100 50  0001 C CNN
+F 1 "GND" H 5205 1177 50  0000 C CNN
+F 2 "" H 5200 1350 50  0001 C CNN
+F 3 "" H 5200 1350 50  0001 C CNN
+	1    5200 1350
+	1    0    0    -1
+$EndComp
+$Comp
+L power:GND #PWR0115
+U 1 1 5B69750E
+P 7500 1600
+F 0 "#PWR0115" H 7500 1350 50  0001 C CNN
+F 1 "GND" H 7505 1427 50  0000 C CNN
+F 2 "" H 7500 1600 50  0001 C CNN
+F 3 "" H 7500 1600 50  0001 C CNN
+	1    7500 1600
+	1    0    0    -1
+$EndComp
+Wire Wire Line
+	7650 1450 7650 1600
+Wire Wire Line
+	7650 1600 7550 1600
+Wire Wire Line
+	7500 1600 7450 1600
+Wire Wire Line
+	7350 1600 7350 1450
+Connection ~ 7500 1600
+Wire Wire Line
+	7450 1450 7450 1600
+Connection ~ 7450 1600
+Wire Wire Line
+	7450 1600 7350 1600
+Wire Wire Line
+	7550 1450 7550 1600
+Connection ~ 7550 1600
+Wire Wire Line
+	7550 1600 7500 1600
+$Comp
+L power:GND #PWR0116
+U 1 1 5B6A7B3B
+P 6950 2350
+F 0 "#PWR0116" H 6950 2100 50  0001 C CNN
+F 1 "GND" H 6955 2177 50  0000 C CNN
+F 2 "" H 6950 2350 50  0001 C CNN
+F 3 "" H 6950 2350 50  0001 C CNN
+	1    6950 2350
+	1    0    0    -1
+$EndComp
+Wire Wire Line
+	6950 2350 6950 2250
+NoConn ~ 800  2150
+NoConn ~ 800  2050
+Wire Wire Line
+	1800 2350 2100 2350
+Wire Wire Line
+	2100 2450 1800 2450
+Text Label 2100 2350 2    60   ~ 0
+A1
+Text Label 2100 2450 2    60   ~ 0
+A2
+Text Label 2850 3250 3    60   ~ 0
+A1
+Text Label 3050 3250 3    60   ~ 0
+A2
+Wire Wire Line
+	2850 3400 2850 3250
+Wire Wire Line
+	3050 3250 3050 3400
 $EndSCHEMATC
