File: layout/arduino-nano-SI5351/ArduinoSpecAn.kicad_pcb (KiCad board)
At the start: 4 copper layers, 60.2 x 50.8 mm, 35 parts, among them J1 SMA, J2 SMA, Q1 Q_NMOS_GSD, Q6 Q_NMOS_GSD, U1 AD8307, U2 LM1117-3.3, U3 LM7301, U4 SI5351, Y1 25MHz

Commit message: Mostly finished
Parts:
- added REF**: WEEE-Logo_5.6x8mm_SilkScreen, Symbol:WEEE-Logo_5.6x8mm_SilkScreen, B.Cu at (155.2, 113.3)
- added REF**: OSHW-Logo_11.4x12mm_SilkScreen, Symbol:OSHW-Logo_11.4x12mm_SilkScreen, B.Cu at (153.4, 123.2)
- R7, R8: value R -> 1kΩ
- moved R8 12.3 mm to (110.7, 131.6), turned to 0 degrees
- moved R7 10.1 mm to (110.7, 133.9), turned to 0 degrees
- moved D1 5.23 mm to (115.1, 133.9), turned to 180 degrees
- moved D2 5.23 mm to (115.1, 131.6), turned to 180 degrees
Connections:
- A1 pad 20: (no net) -> /A1
- A1 pad 21: (no net) -> /A2
- A1 pad 7: Net-(A1-Pad7) -> (no net)
- A1 pad 8: Net-(A1-Pad8) -> (no net)
- D1 pad 1: Net-(A1-Pad8) -> GND
- D2 pad 1: Net-(A1-Pad7) -> GND
- R7 pad 1: Net-(D1-Pad2) -> /A2
- R7 pad 2: GND -> Net-(D1-Pad2)
- R8 pad 1: Net-(D2-Pad2) -> /A1
- R8 pad 2: GND -> Net-(D2-Pad2)
Routing:
- net +5V: track 64.2 -> 101.2 mm, vias 0 -> 2
- net /A1: track 0.00 -> 33.1 mm, vias 0 -> 1
- net /A2: track 0.00 -> 32.9 mm, vias 0 -> 1
- net Net-(A1-Pad7): track 30.5 -> 0.00 mm, vias 1 -> 0
- net Net-(A1-Pad8): track 30.1 -> 0.00 mm, vias 1 -> 0
- net Net-(D2-Pad2): track 15.1 -> 2.38 mm
- net GND: track 292.0 -> 282.3 mm, vias 57 -> 54
- net Net-(D1-Pad2): track 8.98 -> 2.38 mm
- net Net-(Q1-Pad3): track 15.4 -> 13.7 mm
- net /SCL: track 44.0 -> 42.7 mm
- net /SDA: track 49.2 -> 48.4 mm
Other:
- board text added: "3.3V"
- board text added: "5V"
- board text added: "Active"
- board text added: "Connected"
- board text added: "GND"
- board text added: "Network Analyzer Rev. 3a"
- board text added: "OpenNetworkAnalyzer Andreas Butti, 2018 https://github.com/andreasb242/OpenNetworkAnalyzer Based on https://hackaday.io/project/10021-arduino-network-analyzer"
- board text removed: "VNA Rev. 3a"

Commit message: Added reworked app
Other:
- copper layers 4 -> 2
- rule trace_min: 0.2032 -> 0.2
Changed lines of the file:
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@@
   (layers
     (0 F.Cu signal)
-    (1 In1.Cu power)
-    (2 In2.Cu power)
     (31 B.Cu signal)
     (32 B.Adhes user)
@@
     (zone_clearance 0.2032)
     (zone_45_only no)
-    (trace_min 0.2032)
+    (trace_min 0.2)
     (via_size 0.5)
     (via_drill 0.3)
@@
     (visible_elements FFFFFE7F)
     (pcbplotparams
-      (layerselection 0x010f0_80000007)
-      (usegerberextensions true)
+      (layerselection 0x01030_ffffffff)
+      (usegerberextensions false)
       (usegerberattributes false)
       (usegerberadvancedattributes false)
@@
       (psa4output false)
       (plotreference true)
-      (plotvalue false)
+      (plotvalue true)
       (plotinvisibletext false)
       (padsonsilk false)
@@
       (drillshape 0)
       (scaleselection 1)
-      (outputdirectory "/Users/cbkillion/Documents/KiCad Projects/ArduinoSpecAn/Gerbers2/"))
+      (outputdirectory "gerber"))
   )
   (net 0 "")
